File: kicad/parasite.kicad_pcb (KiCad board)
At the start: 2 copper layers, 22 x 126.4 mm, 31 parts, among them Q1 MMBT3906, Q4 Q_Photo_NPN, SW1 B3U-1000P, U1 E73-2G4M08S1C, U2 SHTC3, Y1 32.768kHz

Commit message: rework
Parts:
- added C5: C, Capacitor_SMD:C_0603_1608Metric, F.Cu at (70.2, 47.6)
- added C6: C, Capacitor_SMD:C_0402_1005Metric, F.Cu at (67.6, 47.4)
- added J2: Conn_01x06, b-parasite:490107670612, F.Cu at (76.5, 81.5)
- added NT1: NetTie_2, NetTie:NetTie-2_SMD_Pad0.5mm, F.Cu at (76.8, 60.8)
- moved TP7 24.5 mm to (58.2, 47.4)
- moved D2 19.2 mm to (58.4, 33.8), turned to -90 degrees
- moved R2 14.3 mm to (58.2, 36.2), turned to -90 degrees
- moved TP3 9.49 mm to (74.4, 48.8), turned to 90 degrees
- moved R10 8.39 mm to (58.2, 38.2), turned to -90 degrees
- moved Q4 8.07 mm to (58.2, 40.8)
- moved TP6 5.84 mm to (60.0, 53.8)
- moved R8 5.25 mm to (75.4, 58.2), turned to 0 degrees
- moved TP4 5.17 mm to (73.5, 45.8)
- moved TP2 3.27 mm to (77.0, 34.0)
- moved C2 3.03 mm to (73.5, 56.0)
- moved C3 2.64 mm to (64.8, 51.8)
- moved TP8 2.16 mm to (77.0, 31.8)
- moved C4 2.04 mm to (67.2, 51.8)
- moved Y1 1.89 mm to (66.0, 49.6)
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Connections:
- U1 pad 24: unconnected-(U1A-GND@3-Pad24) -> GND
Routing:
- net SWDCLK: track 6.42 -> 52.3 mm, vias 2 -> 1
- net SWDIO: track 4.18 -> 46.1 mm
- net Net-(J2-Pin_2): track 0.00 -> 23.9 mm, vias 0 -> 1
- net GND: track 22.2 -> 4.09 mm, vias 29 -> 46
- net LED: track 16.9 -> 2.84 mm, vias 2 -> 0
- net RST: track 11.9 -> 4.18 mm, vias 2 -> 0
- net PHOTO_OUT: track 11.5 -> 3.79 mm
- net PHOTO_V: track 8.72 -> 2.71 mm
- net Net-(U1B-P0.01/XL2): track 11.1 -> 7.32 mm
- net Net-(U1B-P0.00/XL1): track 10.2 -> 7.27 mm
- net PWM: track 20.1 -> 17.3 mm
- net SDA: track 24.5 -> 21.7 mm, vias 2 -> 0
- net Net-(D2-A): track 3.51 -> 1.31 mm
- net SENS_OUT: track 38.5 -> 37.4 mm, vias 2 -> 0
- net 0.10: track 4.71 -> 3.62 mm
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Other:
- board text removed: "b-parasite 2.0.0 rbaron.net"
