File: kicad/parasite.kicad_sch (KiCad schematic)
At the start: 29 parts, among them Q1 MMBT3906, Q4 Q_Photo_NPN, SW1 B3U-1000P, U1 E73-2G4M08S1C, U2 SHTC3, Y1 32.768kHz

Commit message: rework
Parts:
- added C5: C, Capacitor_SMD:C_0603_1608Metric, symbol Device:C
- added C6: C, Capacitor_SMD:C_0402_1005Metric, symbol Device:C
- added J2: Conn_01x06, b-parasite:490107670612, symbol Connector_Generic:Conn_01x06
- added NT1: NetTie_2, NetTie:NetTie-2_SMD_Pad0.5mm, symbol Device:NetTie_2
- Q4: PN (none) -> IN-S63DTLS
- Y1: PN (none) -> ABS07-32.768KHZ-T
Connections:
- net +3V0: now also C5.1, C6.1, J2.6 (Pin_6), NT1.2
- net GND: now also U1.24 (GND@3), C5.2, C6.2, J2.1 (Pin_1), J2.3 (Pin_3)
- net SWDCLK: now also J2.4 (Pin_4)
- net SWDIO: now also J2.5 (Pin_5)
- new net: J2.2 (Pin_2), NT1.1
- no-connect marks 25 -> 24
Other:
- moved on the sheet: BT1
